File: KICAD_files/RocketBoard/RocketBoard.kicad_pcb (KiCad board)
At the start: 2 copper layers, 49.2 x 108.1 mm, 16 parts, among them J5 PassiveBuzzer, SW2 ON/OFF, U1 RPI-Pico, U2 L7805, U3 ESP32-CAM

Commit message: bro
Parts:
- J5: footprint Buzzer_Beeper:MagneticBuzzer_Kobitone_254-EMB73-RO -> Buzzer_Beeper:Buzzer_TDK_PS1240P02BT_D12.2mm_H6.5mm
- SW1: renamed from CAM RST
- U1: footprint RpiPico:RPi_Pico_SMD_TH -> MCU_RaspberryPi_and_Boards:RPi_Pico_SMD_TH_2
- moved J5 41.3 mm to (138.4, 97.3), turned to 180 degrees
- renumbered BATT to BATT_IN1
Connections:
- JST_Relay1 pad 1: GND -> Net-(JST_Relay1-Pin_1)
- JST_Relay1 pad 2: Net-(JST_Relay1-Pin_2) -> +5V
- JST_Relay1 pad 3: +5V -> GND
- U1 pad 16: unconnected-(U1-GPIO12-Pad16) -> Net-(J5-Pin_2)
- U1 pad 24: Net-(JST_Relay1-Pin_2) -> Net-(JST_Relay1-Pin_1)
- U1 pad 4: Net-(J5-Pin_2) -> unconnected-(U1-GPIO2-Pad4)
Routing:
- net Net-(JST_Relay1-Pin_2): track 28.8 -> 0.00 mm
- net Net-(JST_Relay1-Pin_1): track 0.00 -> 26.6 mm
- net GND: track 151.5 -> 160.7 mm
- net +5V: track 178.0 -> 181.4 mm
- net Net-(J5-Pin_2): track 11.1 -> 13.1 mm
Other:
- board text added: "4.7K"
- board text removed: "Passive Buzzer"

Commit message: bro
Parts:
- removed JST_Relay1: JST_Relay, Connector_JST:JST_EH_S3B-EH_1x03_P2.50mm_Horizontal
- added D1: 1N4004, Diode_THT:D_A-405_P7.62mm_Horizontal, F.Cu at (127.9, 143.5)
- added D2: RelayLED, LED_THT:LED_D3.0mm, F.Cu at (112.8, 47.8)
- added D3: 1N4004, Diode_THT:D_A-405_P7.62mm_Horizontal, F.Cu at (107.7, 43.7)
- added J1: Relay_OUT, TerminalBlock:TerminalBlock_bornier-2_P5.08mm, F.Cu at (108.7, 37.6)
- added K1: SRD-05VDC-SL-C, Relay5V:RELAY_SRD-05VDC-SL-C, F.Cu at (126.6, 41.7)
- added Q1: 2N2222, Package_TO_SOT_THT:TO-92, F.Cu at (107.1, 48.8)
- added R3: 150, Resistor_THT:R_Axial_DIN0207_L6.3mm_D2.5mm_P10.16mm_Horizontal, F.Cu at (100.6, 41.1)
- SW2: footprint SS2D10:SS12D10 -> SwitchMini:Schiebeschalter SS-12D00
- moved U2 48.9 mm to (139.4, 45.4), turned to 0 degrees
- moved SW2 45.9 mm to (141.6, 39.6), turned to 180 degrees
- moved BATT_IN1 44.3 mm to (141.5, 35.3), turned to 90 degrees
- moved LORA_Socket1 27.1 mm to (118.0, 74.8)
- moved SW1 11.9 mm to (102.7, 60.7)
- moved REF** 9.96 mm to (102.4, 36.8)
- moved U3 8.15 mm to (122.7, 64.1)
- moved R1 5.30 mm to (114.2, 90.6), turned to 90 degrees
- moved R2 4.62 mm to (110.6, 90.6), turned to 90 degrees
Connections:
- BNO08X1 pad 1: GND -> +5V
- BNO08X1 pad 2: +5V -> GND
- U1 pad 39: +5V -> Net-(D1-K)
Routing:
- net GND: track 160.7 -> 199.0 mm
- net Net-(D2-A): track 26.6 -> 63.9 mm
- net Net-(J1-Pin_1): track 0.00 -> 28.2 mm
- net Net-(D3-A): track 0.00 -> 26.3 mm
- net Net-(D1-K): track 0.00 -> 24.3 mm
- net Net-(D2-K): track 0.00 -> 23.7 mm
- net Net-(LORA_Socket1-Pin_3): track 40.3 -> 23.3 mm
- net Net-(LORA_Socket1-Pin_4): track 37.3 -> 24.0 mm
- net +5V: track 181.4 -> 194.3 mm
- net +3.3V: track 60.9 -> 48.4 mm
- net Net-(U1-GPIO7): track 78.4 -> 67.6 mm
- net Net-(BATT_IN1-Pin_2): track 24.2 -> 15.6 mm
- net Net-(J1-Pin_2): track 0.00 -> 6.41 mm
- net Net-(Q1-B): track 0.00 -> 5.53 mm
- net Net-(BATT_IN1-Pin_1): track 8.50 -> 5.41 mm
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Other:
- board size 49.2 x 108.1 mm -> 49.2 x 117.6 mm
- board text removed: "L7805"

Commit message: kikad works
Parts:
- added Pyro1: Pyro2, TerminalBlock:TerminalBlock_bornier-2_P5.08mm, F.Cu at (133.2, 37.8)
- D2: value RelayLED -> RedLED
- J1: value Relay_OUT -> GY-BME-280 Barometer; footprint TerminalBlock:TerminalBlock_bornier-2_P5.08mm -> Connector_PinHeader_2.54mm:PinHeader_1x04_P2.54mm_Vertical; moved to B.Cu
- J5: value PassiveBuzzer -> Buzzer
- moved J1 59.7 mm to (138.8, 89.2)
- moved REF** 41.9 mm to (144.3, 37.5)
- moved BATT_IN1 9.88 mm to (142.9, 45.1)
- moved R1 9.14 mm to (105.0, 90.7)
- moved R2 9.14 mm to (101.5, 90.7)
- moved SW2 8.47 mm to (135.6, 45.6)
- moved D2 7.48 mm to (105.7, 45.5)
- moved D3 7.27 mm to (100.8, 41.3)
- moved U2 6.22 mm to (139.4, 51.6)
- moved K1 6.10 mm to (120.5, 41.8)
- moved Q1 5.99 mm to (106.6, 54.7)
- moved R3 4.57 mm to (100.7, 45.7)
- moved SW1 4.57 mm to (102.7, 65.3)
- moved D1 0.89 mm to (128.8, 143.5)
Connections:
- net Net-(BATT_IN1-Pin_2) renamed WIRE
- J1 pad 1: Net-(J1-Pin_1) -> +3.3V
- J1 pad 2: Net-(J1-Pin_2) -> GND
- K1 pad COM: Net-(J1-Pin_2) -> GND
- K1 pad NC: Net-(J1-Pin_1) -> unconnected-(K1-PadNC)
- K1 pad NO: unconnected-(K1-PadNO) -> Net-(Pyro1-Pin_1)
- U1 pad 19: unconnected-(U1-GPIO14-Pad19) -> Net-(J1-Pin_4)
- U1 pad 20: unconnected-(U1-GPIO15-Pad20) -> Net-(J1-Pin_3)
Routing:
- net +3.3V: track 48.4 -> 132.7 mm
- net Net-(J1-Pin_3): track 0.00 -> 31.2 mm
- net Net-(J1-Pin_1): track 28.2 -> 0.00 mm
- net Net-(J1-Pin_4): track 0.00 -> 24.0 mm
- net +5V: track 194.3 -> 216.7 mm
- net Net-(D2-K): track 23.7 -> 5.05 mm
- net Net-(Pyro1-Pin_1): track 0.00 -> 12.7 mm
- net Net-(D2-A): track 63.9 -> 75.6 mm
- net GND: track 199.0 -> 209.0 mm
- net Net-(LORA_Socket1-Pin_3): track 23.3 -> 32.3 mm
- net Net-(LORA_Socket1-Pin_4): track 24.0 -> 31.7 mm
- net Net-(J1-Pin_2): track 6.41 -> 0.00 mm
- net Net-(JST_GPS1-Pin_3): track 27.1 -> 21.9 mm
- net WIRE: track 15.6 -> 20.3 mm
- net Net-(U3-GND@3): track 8.56 -> 10.4 mm
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Other:
- board text added: "OFF/ON"

Commit message: hhbh
Parts:
- removed LORA_Socket1: LORA_Socket, Connector_PinSocket_2.54mm:PinSocket_1x07_P2.54mm_Vertical
- removed R2: 4.7K, Resistor_THT:R_Axial_DIN0207_L6.3mm_D2.5mm_P10.16mm_Horizontal
- removed REF** (x3): MountingHole_2.2mm_M2, MountingHole:MountingHole_2.2mm_M2
- added H1: MountingHole, MountingHole:MountingHole_2.1mm, F.Cu at (146.5, 148.0)
- added H2: MountingHole, MountingHole:MountingHole_2.1mm, F.Cu at (147.0, 35.0)
- added H3: MountingHole, MountingHole:MountingHole_2.1mm, F.Cu at (102.0, 35.0)
- added H4: MountingHole, MountingHole:MountingHole_2.1mm, F.Cu at (101.5, 148.0)
- added SW3: ON/OFF, roba_mia:Schiebeschalter SS-12D00, F.Cu at (102.5, 83.5)
- BATT1: renamed from BATT_IN1; value BATT_IN -> ~
- J5: value Buzzer -> PassiveBuzzer; footprint Buzzer_Beeper:Buzzer_TDK_PS1240P02BT_D12.2mm_H6.5mm -> roba_mia:myBuzzer
- K1: footprint Relay5V:RELAY_SRD-05VDC-SL-C -> roba_mia:ssr-41FDA
- Pyro1: value Pyro2 -> ~
- R1: value 4.7K -> 10K omh; footprint Resistor_THT:R_Axial_DIN0207_L6.3mm_D2.5mm_P10.16mm_Horizontal -> Resistor_THT:R_Axial_DIN0204_L3.6mm_D1.6mm_P5.08mm_Horizontal
- U1: footprint MCU_RaspberryPi_and_Boards:RPi_Pico_SMD_TH_2 -> raspberry pi pico:RPi_Pico_SMD_TH
- moved D3 23.5 mm to (123.8, 36.0), turned to 180 degrees
- moved Q1 16.5 mm to (110.0, 38.5), turned to 90 degrees
- moved J1 13.0 mm to (147.5, 79.5), turned to 90 degrees
- moved SW2 10.5 mm to (142.0, 54.0), turned to 0 degrees
- moved J5 6.32 mm to (143.8, 94.0)
- moved R3 6.29 mm to (103.0, 51.6), turned to 90 degrees
- moved BATT1 6.11 mm to (138.9, 49.8), turned to 180 degrees
- moved K1 5.99 mm to (125.7, 44.7)
- moved U2 5.90 mm to (139.4, 57.5)
- moved SW1 4.74 mm to (103.0, 70.0)
- moved Pyro1 3.91 mm to (136.8, 36.2), turned to 180 degrees
- moved D2 2.92 mm to (108.2, 44.0)
- moved U3 2.76 mm to (120.4, 62.6)
- moved BNO08X1 2.06 mm to (134.5, 106.3)
- moved JST_GPS1 1.80 mm to (142.0, 134.4)
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Connections:
- net Net-(BATT_IN1-Pin_1) renamed /battGNDpreSwitch
- net Net-(D1-K) renamed /5V 
- net Net-(D3-A) renamed /Relè_GND_signal
- net Net-(U3-GND@3) renamed /esp32_GND
- net WIRE renamed /batt_vcc
- K1 pad COM: GND -> /batt_GND_after_relè
- K1 pad NO: Net-(Pyro1-Pin_1) -> GND
- Pyro1 pad 1: Net-(Pyro1-Pin_1) -> /batt_GND_after_relè
- R1 pad 1: +3.3V -> GND
- R1 pad 2: Net-(LORA_Socket1-Pin_3) -> Net-(SW3-B)
- U1 pad 10: Net-(U1-GPIO7) -> unconnected-(U1-GPIO7-Pad10)
- U1 pad 12: unconnected-(U1-GPIO9-Pad12) -> Net-(SW3-B)
- U1 pad 21: Net-(LORA_Socket1-Pin_3) -> Net-(U1-GPIO16)
- U1 pad 22: Net-(LORA_Socket1-Pin_4) -> Net-(U1-GPIO17)
- U1 pad 28: GND -> unconnected-(U1-GND-Pad28)
- U1 pad 30: unconnected-(U1-RUN-Pad30) -> GND
- U1 pad 8: unconnected-(U1-GND-Pad8) -> GND
- U3 pad P$2: unconnected-(U3-GPIO1-PadP$2) -> Net-(U1-GPIO17)
- U3 pad P$3: Net-(U1-GPIO7) -> Net-(U1-GPIO16)
Routing:
- net Net-(U1-GPIO7): track 67.6 -> 0.00 mm
- net +5V: track 216.7 -> 158.6 mm
- net Net-(U1-GPIO17): track 0.00 -> 49.5 mm
- net Net-(U1-GPIO16): track 0.00 -> 40.5 mm
- net GND: track 209.0 -> 168.8 mm
- net Net-(SW3-B): track 0.00 -> 39.7 mm
- net Net-(LORA_Socket1-Pin_3): track 32.3 -> 0.00 mm
- net Net-(LORA_Socket1-Pin_4): track 31.7 -> 0.00 mm
- net +3.3V: track 132.7 -> 101.5 mm, vias 0 -> 1
- net /batt_vcc: track 20.3 -> 36.7 mm
- net Net-(Pyro1-Pin_1): track 12.7 -> 0.00 mm
- net Net-(J1-Pin_4): track 24.0 -> 36.7 mm
- net /Relè_GND_signal: track 25.0 -> 14.8 mm
- net Net-(D2-A): track 75.6 -> 66.1 mm
- net /batt_GND_after_relè: track 0.00 -> 6.53 mm
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- added copper zone on B.Cu, net /batt_vcc
- added copper zone on B.Cu, net GND
Other:
- board size 49.2 x 117.6 mm -> 51.7 x 119.5 mm
- board text added: "10K"
- board text added: "DATA"
- board text added: "Made by Simone Cargnin"
- board text added: "ON/OFF"
- board text added: "SSR-41FDA"
- board text removed: "4.7K"
- board text removed: "Designed by Lud"
- board text removed: "Made in collaboration with Simone Cargnin & Vittorio Sedda"
- board text removed: "Rocket-Control Board"
- board text removed: "Sbirro guarda un po' più in la del tuo binocolo Non c'è una scelta se i bisogni te li impongono"
