File: KICAD_files/RocketBoard/RocketBoard.kicad_sch (KiCad schematic)
At the start: 17 parts, among them J5 PassiveBuzzer, SW1 RESET, SW2 ON/OFF, U1 RPI-Pico, U2 L7805, U3 ESP32-CAM

Commit message: bro
Parts:
- J5: footprint Buzzer_Beeper:MagneticBuzzer_Kobitone_254-EMB73-RO -> Buzzer_Beeper:Buzzer_TDK_PS1240P02BT_D12.2mm_H6.5mm
- U1: footprint RpiPico:RPi_Pico_SMD_TH -> MCU_RaspberryPi_and_Boards:RPi_Pico_SMD_TH_2
Connections:
- net +5V: now also JST_Relay1.2 (Pin_2); no longer JST_Relay1.3 (Pin_3)
- net GND: now also JST_Relay1.3 (Pin_3); no longer JST_Relay1.1 (Pin_1)
- net at U1.16 (GPIO12): now also J5.2 (Pin_2)
- net at U1.24 (GPIO18): now also JST_Relay1.1 (Pin_1); no longer JST_Relay1.2 (Pin_2)
- net at U1.4 (GPIO2): no longer J5.2 (Pin_2)
Other:
- note removed: "Normally Closed Switch SMD"
- note removed: "SS12D10"
Changed lines of the file:
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@@
   (junction (at 156.21 115.57) (diameter 0) (color 0 0 0 0)
   )
+  (junction (at 144.78 97.79) (diameter 0) (color 0 0 0 0)
+  )
   (junction (at 133.35 43.18) (diameter 0) (color 0 0 0 0)
   )
-  (junction (at 144.78 97.79) (diameter 0) (color 0 0 0 0)
-  )
   (wire (pts (xy 156.21 114.3) (xy 156.21 115.57))
     (stroke (width 0) (type default))
@@
     (stroke (width 0) (type default))
   )
+  (wire (pts (xy 147.32 92.71) (xy 151.13 92.71))
+    (stroke (width 0) (type default))
+  )
+  (wire (pts (xy 93.98 72.39) (xy 93.98 86.36))
+    (stroke (width 0) (type default))
+  )
   (wire (pts (xy 147.32 107.95) (xy 137.16 107.95))
     (stroke (width 0) (type default))
   )
-  (wire (pts (xy 93.98 74.93) (xy 101.6 74.93))
-    (stroke (width 0) (type default))
-  )
-  (wire (pts (xy 144.78 92.71) (xy 144.78 97.79))
+  (wire (pts (xy 97.79 86.36) (xy 93.98 86.36))
     (stroke (width 0) (type default))
   )
@@
     (stroke (width 0) (type default))
   )
+  (wire (pts (xy 97.79 86.36) (xy 97.79 105.41))
+    (stroke (width 0) (type default))
+  )
+  (wire (pts (xy 83.82 72.39) (xy 93.98 72.39))
+    (stroke (width 0) (type default))
+  )
   (wire (pts (xy 137.16 69.85) (xy 139.7 69.85))
     (stroke (width 0) (type default))
@@
     (stroke (width 0) (type default))
   )
-  (wire (pts (xy 83.82 72.39) (xy 93.98 72.39))
-    (stroke (width 0) (type default))
-  )
   (wire (pts (xy 186.69 110.49) (xy 184.15 110.49))
     (stroke (width 0) (type default))
@@
     (stroke (width 0) (type default))
   )
+  (wire (pts (xy 97.79 105.41) (xy 101.6 105.41))
+    (stroke (width 0) (type default))
+  )
   (wire (pts (xy 97.79 97.79) (xy 101.6 97.79))
     (stroke (width 0) (type default))
@@
     (stroke (width 0) (type default))
   )
-  (wire (pts (xy 151.13 95.25) (xy 147.32 95.25))
-    (stroke (width 0) (type default))
-  )
   (wire (pts (xy 101.6 82.55) (xy 88.9 82.55))
     (stroke (width 0) (type default))
   )
-  (wire (pts (xy 147.32 95.25) (xy 147.32 107.95))
+  (wire (pts (xy 147.32 92.71) (xy 147.32 107.95))
     (stroke (width 0) (type default))
   )
@@
     (stroke (width 0) (type default))
   )
-  (wire (pts (xy 93.98 72.39) (xy 93.98 74.93))
-    (stroke (width 0) (type default))
-  )
   (wire (pts (xy 186.69 123.19) (xy 184.15 123.19))
     (stroke (width 0) (type default))
@@
     (stroke (width 0) (type default))
   )
-  (wire (pts (xy 151.13 92.71) (xy 144.78 92.71))
-    (stroke (width 0) (type default))
-  )
   (wire (pts (xy 69.85 36.83) (xy 68.58 36.83))
     (stroke (width 0) (type default))
@@
   )
   (wire (pts (xy 137.16 113.03) (xy 140.97 113.03))
+    (stroke (width 0) (type default))
+  )
+  (wire (pts (xy 144.78 97.79) (xy 151.13 97.79))
     (stroke (width 0) (type default))
   )
@@
     (effects (font (size 1.27 1.27)) (justify right bottom))
   )
-  (text "Normally Closed\nSwitch SMD\n" (at 40.64 135.89 90)
-    (effects (font (size 1.27 1.27) bold italic) (justify left bottom))
-  )
   (text "RX" (at 71.12 85.09 0)
     (effects (font (size 1.27 1.27)) (justify left bottom))
@@
   (text "RX" (at 96.52 85.09 0)
     (effects (font (size 1.27 1.27)) (justify left bottom))
-  )
-  (text "SS12D10" (at 132.08 27.94 0)
-    (effects (font (size 1.27 1.27) (thickness 0.254) bold italic) (justify right bottom))
   )
   (text "TX" (at 185.42 115.57 0)
@@
       (effects (font (size 1.27 1.27)))
     )
-    (property "Footprint" "RpiPico:RPi_Pico_SMD_TH" (at 119.38 91.44 90)
+    (property "Footprint" "MCU_RaspberryPi_and_Boards:RPi_Pico_SMD_TH_2" (at 119.38 91.44 90)
       (effects (font (size 1.27 1.27)) hide)
     )
@@
     )
   )
-  (symbol (lib_id "power:+5V") (at 151.13 97.79 90) (unit 1)
+  (symbol (lib_id "power:+5V") (at 151.13 95.25 90) (unit 1)
     (in_bom yes) (on_board yes) (dnp no)
-    (property "Reference" "#PWR06" (at 154.94 97.79 0)
-      (effects (font (size 1.27 1.27)) hide)
-    )
-    (property "Value" "+5V" (at 151.13 100.33 90)
-      (effects (font (size 1.27 1.27)) (justify left))
-    )
-    (property "Footprint" "" (at 151.13 97.79 0)
-      (effects (font (size 1.27 1.27)) hide)
-    )
-    (property "Datasheet" "" (at 151.13 97.79 0)
+    (property "Reference" "#PWR06" (at 154.94 95.25 0)
+      (effects (font (size 1.27 1.27)) hide)
+    )
+    (property "Value" "+5V" (at 146.05 95.25 90)
+      (effects (font (size 1.27 1.27)) (justify left))
+    )
+    (property "Footprint" "" (at 151.13 95.25 0)
+      (effects (font (size 1.27 1.27)) hide)
+    )
+    (property "Datasheet" "" (at 151.13 95.25 0)
       (effects (font (size 1.27 1.27)) hide)
     )
@@
       (effects (font (size 1.27 1.27)) (justify left))
     )
-    (property "Footprint" "Buzzer_Beeper:MagneticBuzzer_Kobitone_254-EMB73-RO" (at 78.74 74.93 0)
-      (effects (font (size 1.27 1.27)) hide)
-    )
+    (property "Footprint" "Buzzer_Beeper:Buzzer_TDK_PS1240P02BT_D12.2mm_H6.5mm" (at 78.74 74.93 0)
+      (effects (font (size 1.27 1.27)) hide)
+    )

Commit message: bro
Parts:
- removed JST_Relay1: JST_Relay, Connector_JST:JST_EH_S3B-EH_1x03_P2.50mm_Horizontal, symbol Connector:Conn_01x03_Socket
- added D1, D3: 1N4004, Diode_THT:D_A-405_P7.62mm_Horizontal, symbol Device:D
- added D2: RelayLED, LED_THT:LED_D3.0mm, symbol Device:LED
- added J1: Relay_OUT, TerminalBlock:TerminalBlock_bornier-2_P5.08mm, symbol Connector:Conn_01x02_Pin
- added K1: SRD-05VDC-SL-C, Relay5V:RELAY_SRD-05VDC-SL-C, symbol SRD-05VDC-SL-C:SRD-05VDC-SL-C
- added Q1: 2N2222, Package_TO_SOT_THT:TO-92, symbol Transistor_BJT:2N2219
- added R3: 150, Resistor_THT:R_Axial_DIN0207_L6.3mm_D2.5mm_P10.16mm_Horizontal, symbol Device:R
- SW2: footprint SS2D10:SS12D10 -> SwitchMini:Schiebeschalter SS-12D00
Connections:
- net +5V: now also BNO08X1.1 (Pin_1), D1.2 (A), D3.1 (K), K1.A2; no longer BNO08X1.2 (Pin_2), U1.39 (VSYS)
- net GND: now also BNO08X1.2 (Pin_2), Q1.3 (C); no longer BNO08X1.1 (Pin_1), U1.42 (GND)
- net at U1.24 (GPIO18): now also D2.2 (A)
- new net: J1.1 (Pin_1), K1.NC
- new net: J1.2 (Pin_2), K1.COM
- new net: D2.1 (K), R3.1
- new net: Q1.2 (B), R3.2
- new net: D1.1 (K), U1.39 (VSYS)
- new net: D3.2 (A), K1.A1, Q1.1 (E)
Other:
- moved on the sheet: J5, JST_GPS1, SW1, U3

Commit message: kikad works
Parts:
- added J1: GY-BME-280 Barometer, Connector_PinHeader_2.54mm:PinHeader_1x04_P2.54mm_Vertical, symbol Connector:Conn_01x04_Socket
- D2: value RelayLED -> RedLED
- Pyro1: renamed from J1; value Relay_OUT -> Pyro2
Connections:
- net +3.3V: now also J1.1 (Pin_1)
- net GND: now also K1.COM, J1.2 (Pin_2)
- net WIRE: now reaches BATT_IN1.2 (Pin_2), U2.1 (IN)
- net WIRE: now also Pyro1.2 (Pin_2)
- net at Pyro1.1 (Pin_1): now also K1.NO; no longer K1.NC
- net at U1.19 (GPIO14): now also J1.4 (Pin_4)
- net at U1.20 (GPIO15): now also J1.3 (Pin_3)
Other:
- moved on the sheet: BATT_IN1, BNO08X1, D1, D2, D3, H1, H2, H3, H4, J5, JST_GPS1, K1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

Commit message: bros
Parts:
- BATT_VCC: renamed from BATT_IN1; value BATT_IN -> BATT_GND
Connections:
- net WIRE: no longer names the net of BATT_VCC.2 (Batt_GND), Pyro1.2 (Pin_2), U2.1 (IN)
Other:
- note added: "battery 2s lipo 7.4V 1A"
- moved on the sheet: BATT_VCC, H1, H2, H3, H4, J1, J5, SW2, U2

Commit message: hhbh
Parts:
- removed LORA_Socket1: LORA_Socket, Connector_PinSocket_2.54mm:PinSocket_1x07_P2.54mm_Vertical, symbol Connector:Conn_01x07_Socket
- removed R2: 4.7K, Resistor_THT:R_Axial_DIN0207_L6.3mm_D2.5mm_P10.16mm_Horizontal, symbol Device:R
- added SW3: ON/OFF, roba_mia:Schiebeschalter SS-12D00, symbol Switch:SW_SPST
- BATT1: renamed from BATT_VCC; value BATT_GND -> ~
- H1, H2, H3, H4: footprint (none) -> MountingHole:MountingHole_2.1mm
- J5: footprint Buzzer_Beeper:Buzzer_TDK_PS1240P02BT_D12.2mm_H6.5mm -> roba_mia:myBuzzer
- K1: footprint Relay5V:RELAY_SRD-05VDC-SL-C -> roba_mia:ssr-41FDA
- Pyro1: value Pyro2 -> ~
- R1: value 4.7K -> 10K omh; footprint Resistor_THT:R_Axial_DIN0207_L6.3mm_D2.5mm_P10.16mm_Horizontal -> Resistor_THT:R_Axial_DIN0204_L3.6mm_D1.6mm_P5.08mm_Horizontal
- U1: footprint MCU_RaspberryPi_and_Boards:RPi_Pico_SMD_TH_2 -> raspberry pi pico:RPi_Pico_SMD_TH
Connections:
- net +3.3V: now also SW3.1 (A); no longer R1.1
- net GND: now also K1.NO, R1.1, U1.30 (RUN), U1.8 (GND); no longer K1.COM, U1.28 (GND)
- net batt_vcc: now reaches BATT1.2 (BATT_VCC), Pyro1.2 (Pin_2), U2.1 (IN)
- net battGNDpreSwitch: now reaches BATT1.1 (BATT_GND), SW2.1 (A)
- net at R1.2: now also U1.12 (GPIO9), SW3.2 (B); no longer U1.21 (GPIO16)
- net batt_GND_after_relè: now reaches Pyro1.1 (Pin_1)
- net batt_GND_after_relè: now also K1.COM; no longer K1.NO
- net at U1.10 (GPIO7): no longer U3.P$3 (GPIO3)
- net at U1.22 (GPIO17): now also U3.P$2 (GPIO1)
- net 5V : now reaches D1.1 (K), U1.39 (VSYS)
- net esp32_GND: now reaches SW1.2, U3.P$10 (GND@3)
- net Relè_GND_signal: now reaches D3.2 (A), K1.A1, Q1.1 (E)
- new net: U1.21 (GPIO16), U3.P$3 (GPIO3)
Other:
- note added: "rx"
- note added: "tx"
- note removed: "AUX"
- note removed: "LORA Module"
- note removed: "M0 M1"
- moved on the sheet: D2, D3, J5, K1, Q1, R3, SW1, SW2, U2, U3
